File: Hardware/Krankenwagen_PCB/Krankenwagen_PCB.kicad_sch (KiCad schematic)
At the start: 3 parts

Commit message: Completed schematic
Parts:
- added H? (x3): 3.5mm Plated Holes, symbol Mechanical:MountingHole
- added H? (x6): 2.8mm Plated Holes, symbol Mechanical:MountingHole
Connections:
- net +12V: now also H?.1, H?.1, H?.1
- net GND: now also H?.2, H?.2, H?.2
- new net: H?.1, H?.1 (x3)
- new net: H?.2, H?.2 (x3)
- new net: H?.3, H?.3 (x3)
Other:
- note added: "12AWG equivalent"
- note added: "12AWG wires from ESC"
- note added: "14AWG equivalent"
- note added: "14AWG wires from ESC"
- note added: "Battery Connections"
- note added: "Holes 70% Larger Than Wires"
- note added: "Motor"
- note added: "Motor ESC"
- note added: "Motor phases"
- note added: "Traces rated for 32A continuous,"
- note added: "Traces rated for 41A continuous,"
- company: (none) -> Missouri S&T Combot Robotics Team - Thomas Francois
- title: (none) -> Krankenwagen ESC & Motor PCB
- moved on the sheet: J?

Commit message: Created solder hole footprints
Other:
- note added: "Castle 1410 BLDC Motors"
Changed lines of the file:
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@@
     (effects (font (size 2.54 2.54)) (justify left bottom))
+  )
+  (text "Castle 1410 BLDC Motors" (at 244.475 60.96 0)
+    (effects (font (size 1.27 1.27) bold italic) (justify left bottom))
   )
   (text "Motor" (at 238.76 97.79 0)
